File: 1wire-4switch/1wire-4switch.kicad_pcb (KiCad board)
At the start: 2 copper layers, 65.5 x 59.4 mm, 18 parts, among them IC1 DS2408S, J1 RJ45, J2 RJ45, K1 CONN_3, K2 CONN_3, P1 CONN_4, P2 CONN_4, P3 CONN_5_V, P4 CONN_4, U1 74HC04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

Commit message: Bring the 4 channel switch module up to date
Signed-off-by: Alastair D'Silva <alastair@d-silva.org>
Other:
- board text added: "©2016 Inferno Embedded"
- board text removed: "©2014 Inferno Embedded"
Changed lines of the file:
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@@
     (visible_elements 7FFFFBFF)
     (pcbplotparams
-      (layerselection 0x00030_80000001)
+      (layerselection 0x010f0_80000001)
       (usegerberextensions true)
       (excludeedgelayer true)
@@
     (effects (font (size 1.5 1.5) (thickness 0.3)))
   )
-  (gr_text "©2014 Inferno Embedded" (at 138.684 121.92 90) (layer F.SilkS)
-    (effects (font (size 1.5 1.5) (thickness 0.3)))
-  )
+  (gr_text "©2016 Inferno Embedded" (at 138.684 121.92 90) (layer F.SilkS)
+    (effects (font (size 1.5 1.5) (thickness 0.3)))
+  )
