File: devices/PiMultichannelMaster/OutputBoard/1wiredriver.sch (KiCad schematic (older format))
At the start: 30 parts, among them Q1 2N7002, Q2 2N7002, Q3 2N7002, Q4 2N7002, Q5 BSS84, Q6 BSS84, Q7 BSS84, Q8 BSS84

Commit message: Add pullups to the PiMultichannelMaster outputboard pullup mosfet
Parts:
- added RP13: 100k, 0603-pack4:0603_Pack4, symbol R_PACK4
Connections:
- net +5V: now also RP13.5 (R4), RP13.6 (R3), RP13.7 (R2), RP13.8 (R1)
- net at C7.2, Q5.1 (G), RP2.1 (P1): now also RP13.4 (P4)
- net at C8.2, Q6.1 (G), RP2.2 (P2): now also RP13.3 (P3)
- net at C9.2, Q7.1 (G), RP2.3 (P3): now also RP13.2 (P2)
- net at C10.2, Q8.1 (G), RP2.4 (P4): now also RP13.1 (P1)
Changed lines of the file:
@@
 Title "1Wire Driver"
 Date "2017-06-13"
-Rev "1.0"
+Rev "1.1"
 Comp "Inferno Embedded"
 Comment1 ""
@@
 P 7300 900
 AR Path="/5943BBDD/5942CA97" Ref="#PWR024"  Part="1"
-AR Path="/5943EE87/5942CA97" Ref="#PWR042"  Part="1"
-F 0 "#PWR042" H 7300 750 50  0001 C CNN
+AR Path="/5943EE87/5942CA97" Ref="#PWR043"  Part="1"
+F 0 "#PWR043" H 7300 750 50  0001 C CNN
 F 1 "+5V" H 7300 1040 50  0000 C CNN
 F 2 "" H 7300 900 50  0000 C CNN
@@
 P 7300 1950
 AR Path="/5943BBDD/5942CA9D" Ref="#PWR025"  Part="1"
-AR Path="/5943EE87/5942CA9D" Ref="#PWR043"  Part="1"
-F 0 "#PWR043" H 7300 1700 50  0001 C CNN
+AR Path="/5943EE87/5942CA9D" Ref="#PWR044"  Part="1"
+F 0 "#PWR044" H 7300 1700 50  0001 C CNN
 F 1 "GND" H 7300 1800 50  0000 C CNN
 F 2 "" H 7300 1950 50  0000 C CNN
@@
 P 8200 900
 AR Path="/5943BBDD/5942CC90" Ref="#PWR026"  Part="1"
-AR Path="/5943EE87/5942CC90" Ref="#PWR044"  Part="1"
-F 0 "#PWR044" H 8200 750 50  0001 C CNN
+AR Path="/5943EE87/5942CC90" Ref="#PWR045"  Part="1"
+F 0 "#PWR045" H 8200 750 50  0001 C CNN
 F 1 "+5V" H 8200 1040 50  0000 C CNN
 F 2 "" H 8200 900 50  0000 C CNN
@@
 P 8200 1950
 AR Path="/5943BBDD/5942CC96" Ref="#PWR027"  Part="1"
-AR Path="/5943EE87/5942CC96" Ref="#PWR045"  Part="1"
-F 0 "#PWR045" H 8200 1700 50  0001 C CNN
+AR Path="/5943EE87/5942CC96" Ref="#PWR046"  Part="1"
+F 0 "#PWR046" H 8200 1700 50  0001 C CNN
 F 1 "GND" H 8200 1800 50  0000 C CNN
 F 2 "" H 8200 1950 50  0000 C CNN
@@
 P 9100 900
 AR Path="/5943BBDD/5942CCFE" Ref="#PWR028"  Part="1"
-AR Path="/5943EE87/5942CCFE" Ref="#PWR046"  Part="1"
-F 0 "#PWR046" H 9100 750 50  0001 C CNN
+AR Path="/5943EE87/5942CCFE" Ref="#PWR047"  Part="1"
+F 0 "#PWR047" H 9100 750 50  0001 C CNN
 F 1 "+5V" H 9100 1040 50  0000 C CNN
 F 2 "" H 9100 900 50  0000 C CNN
@@
 P 9100 1950
 AR Path="/5943BBDD/5942CD04" Ref="#PWR029"  Part="1"
-AR Path="/5943EE87/5942CD04" Ref="#PWR047"  Part="1"
-F 0 "#PWR047" H 9100 1700 50  0001 C CNN
+AR Path="/5943EE87/5942CD04" Ref="#PWR048"  Part="1"
+F 0 "#PWR048" H 9100 1700 50  0001 C CNN
 F 1 "GND" H 9100 1800 50  0000 C CNN
 F 2 "" H 9100 1950 50  0000 C CNN
@@
 P 10000 900
 AR Path="/5943BBDD/5942CD14" Ref="#PWR030"  Part="1"
-AR Path="/5943EE87/5942CD14" Ref="#PWR048"  Part="1"
-F 0 "#PWR048" H 10000 750 50  0001 C CNN
+AR Path="/5943EE87/5942CD14" Ref="#PWR049"  Part="1"
+F 0 "#PWR049" H 10000 750 50  0001 C CNN
 F 1 "+5V" H 10000 1040 50  0000 C CNN
 F 2 "" H 10000 900 50  0000 C CNN
@@
 P 10000 1950
 AR Path="/5943BBDD/5942CD1A" Ref="#PWR031"  Part="1"
-AR Path="/5943EE87/5942CD1A" Ref="#PWR049"  Part="1"
-F 0 "#PWR049" H 10000 1700 50  0001 C CNN
+AR Path="/5943EE87/5942CD1A" Ref="#PWR050"  Part="1"
+F 0 "#PWR050" H 10000 1700 50  0001 C CNN
 F 1 "GND" H 10000 1800 50  0000 C CNN
 F 2 "" H 10000 1950 50  0000 C CNN
@@
 P 6350 800
 AR Path="/5943BBDD/5942DBEB" Ref="#PWR032"  Part="1"
-AR Path="/5943EE87/5942DBEB" Ref="#PWR050"  Part="1"
-F 0 "#PWR050" H 6350 650 50  0001 C CNN
+AR Path="/5943EE87/5942DBEB" Ref="#PWR051"  Part="1"
+F 0 "#PWR051" H 6350 650 50  0001 C CNN
 F 1 "+5V" H 6350 940 50  0000 C CNN
 F 2 "" H 6350 800 50  0000 C CNN
@@
 P 6350 1700
 AR Path="/5943BBDD/5942DD2A" Ref="#PWR033"  Part="1"
-AR Path="/5943EE87/5942DD2A" Ref="#PWR051"  Part="1"
-F 0 "#PWR051" H 6350 1550 50  0001 C CNN
+AR Path="/5943EE87/5942DD2A" Ref="#PWR052"  Part="1"
+F 0 "#PWR052" H 6350 1550 50  0001 C CNN
 F 1 "+5V" H 6350 1840 50  0000 C CNN
 F 2 "" H 6350 1700 50  0000 C CNN
@@
 P 6350 2600
 AR Path="/5943BBDD/5942DF27" Ref="#PWR034"  Part="1"
-AR Path="/5943EE87/5942DF27" Ref="#PWR052"  Part="1"
-F 0 "#PWR052" H 6350 2450 50  0001 C CNN
+AR Path="/5943EE87/5942DF27" Ref="#PWR053"  Part="1"
+F 0 "#PWR053" H 6350 2450 50  0001 C CNN
 F 1 "+5V" H 6350 2740 50  0000 C CNN
 F 2 "" H 6350 2600 50  0000 C CNN
@@
 P 6350 3500
 AR Path="/5943BBDD/5942DF40" Ref="#PWR035"  Part="1"
-AR Path="/5943EE87/5942DF40" Ref="#PWR053"  Part="1"
-F 0 "#PWR053" H 6350 3350 50  0001 C CNN
+AR Path="/5943EE87/5942DF40" Ref="#PWR054"  Part="1"
+F 0 "#PWR054" H 6350 3350 50  0001 C CNN
 F 1 "+5V" H 6350 3640 50  0000 C CNN
 F 2 "" H 6350 3500 50  0000 C CNN
@@
 P 8750 4100
 AR Path="/5943BBDD/5942E7BC" Ref="#PWR036"  Part="1"
-AR Path="/5943EE87/5942E7BC" Ref="#PWR054"  Part="1"
-F 0 "#PWR054" H 8750 3950 50  0001 C CNN
+AR Path="/5943EE87/5942E7BC" Ref="#PWR055"  Part="1"
+F 0 "#PWR055" H 8750 3950 50  0001 C CNN
 F 1 "+5V" H 8750 4240 50  0000 C CNN
 F 2 "" H 8750 4100 50  0000 C CNN
@@
 P 9400 4500
 AR Path="/5943BBDD/5942F5D4" Ref="#PWR037"  Part="1"
-AR Path="/5943EE87/5942F5D4" Ref="#PWR055"  Part="1"
-F 0 "#PWR055" H 9400 4250 50  0001 C CNN
+AR Path="/5943EE87/5942F5D4" Ref="#PWR056"  Part="1"
+F 0 "#PWR056" H 9400 4250 50  0001 C CNN
 F 1 "GND" H 9400 4350 50  0000 C CNN
 F 2 "" H 9400 4500 50  0000 C CNN
@@
 P 3000 1500
 AR Path="/5943BBDD/59430490" Ref="#PWR038"  Part="1"
-AR Path="/5943EE87/59430490" Ref="#PWR056"  Part="1"
-F 0 "#PWR056" H 3000 1250 50  0001 C CNN
+AR Path="/5943EE87/59430490" Ref="#PWR057"  Part="1"
+F 0 "#PWR057" H 3000 1250 50  0001 C CNN
 F 1 "GND" H 3000 1350 50  0000 C CNN
 F 2 "" H 3000 1500 50  0000 C CNN
@@
 P 3000 2450
 AR Path="/5943BBDD/59430CBD" Ref="#PWR039"  Part="1"
-AR Path="/5943EE87/59430CBD" Ref="#PWR057"  Part="1"
-F 0 "#PWR057" H 3000 2200 50  0001 C CNN
+AR Path="/5943EE87/59430CBD" Ref="#PWR058"  Part="1"
+F 0 "#PWR058" H 3000 2200 50  0001 C CNN
 F 1 "GND" H 3000 2300 50  0000 C CNN
 F 2 "" H 3000 2450 50  0000 C CNN
@@
 P 3000 3450
 AR Path="/5943BBDD/59430E24" Ref="#PWR040"  Part="1"
-AR Path="/5943EE87/59430E24" Ref="#PWR058"  Part="1"
-F 0 "#PWR058" H 3000 3200 50  0001 C CNN
+AR Path="/5943EE87/59430E24" Ref="#PWR059"  Part="1"
+F 0 "#PWR059" H 3000 3200 50  0001 C CNN
 F 1 "GND" H 3000 3300 50  0000 C CNN
 F 2 "" H 3000 3450 50  0000 C CNN
@@
 P 3000 4400
 AR Path="/5943BBDD/59430E3D" Ref="#PWR041"  Part="1"
-AR Path="/5943EE87/59430E3D" Ref="#PWR059"  Part="1"
-F 0 "#PWR059" H 3000 4150 50  0001 C CNN
+AR Path="/5943EE87/59430E3D" Ref="#PWR060"  Part="1"
+F 0 "#PWR060" H 3000 4150 50  0001 C CNN
 F 1 "GND" H 3000 4250 50  0000 C CNN
 F 2 "" H 3000 4400 50  0000 C CNN
@@
 	10250 1550 10250 1500
 Connection ~ 10250 1500
+$Comp
+L R_PACK4 RP13
+U 1 1 59899A81
+P 5050 1150
+AR Path="/5943BBDD/59899A81" Ref="RP13"  Part="1"
+AR Path="/5943EE87/59899A81" Ref="RP14"  Part="1"
+F 0 "RP13" H 5050 1600 50  0000 C CNN
+F 1 "100k" H 5050 1100 50  0000 C CNN
+F 2 "0603-pack4:0603_Pack4" H 5050 1150 50  0001 C CNN
+F 3 "" H 5050 1150 50  0000 C CNN
+	1    5050 1150
+	-1   0    0    1
+$EndComp
+Wire Wire Line
+	5250 1500 5300 1500
+Wire Wire Line
+	5300 1500 5300 2200
+Connection ~ 5300 2200
+Wire Wire Line
+	5250 1400 5350 1400
+Wire Wire Line
+	5350 1400 5350 2100
+Connection ~ 5350 2100
+Wire Wire Line
+	5250 1300 5400 1300
+Wire Wire Line
+	5400 1300 5400 2000
+Connection ~ 5400 2000
+Wire Wire Line
+	5250 1200 5450 1200
+Wire Wire Line
+	5450 1200 5450 1900
+Connection ~ 5450 1900
+$Comp
+L +5V #PWR042
+U 1 1 59899E71
+P 4750 800
+AR Path="/5943BBDD/59899E71" Ref="#PWR042"  Part="1"
+AR Path="/5943EE87/59899E71" Ref="#PWR061"  Part="1"
+F 0 "#PWR061" H 4750 650 50  0001 C CNN
+F 1 "+5V" H 4750 940 50  0000 C CNN
+F 2 "" H 4750 800 50  0000 C CNN
+F 3 "" H 4750 800 50  0000 C CNN
+	1    4750 800
+	1    0    0    -1
+$EndComp
+Wire Wire Line
+	4750 800  4750 1500
+Wire Wire Line
+	4750 1500 4850 1500
+Wire Wire Line
+	4850 1400 4750 1400
+Connection ~ 4750 1400
+Wire Wire Line
+	4850 1300 4750 1300
+Connection ~ 4750 1300
+Wire Wire Line
+	4850 1200 4750 1200
+Connection ~ 4750 1200
 $EndSCHEMATC
