File: devices/Inline_SSR/Inline_SSR.kicad_pcb (KiCad board)
At the start: 2 copper layers, 17.1 x 30.5 mm, 4 parts, among them J1 JACK_STEREO, P1 CONN_01X02, U1 G3MB_SSR

Commit message: Big cleanup/upgrade of Kicad files
Routing:
- net Net-(P1-Pad1): track 6.76 -> 13.5 mm
Other:
- outline, holes or cut-outs redrawn
Changed lines of the file:
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@@
-(kicad_pcb (version 4) (host pcbnew 4.0.4-stable)
+(kicad_pcb (version 20171130) (host pcbnew "(5.0.1)-3")
   (general
-    (links 8)
-    (no_connects 0)
-    (area 144.704999 77.451 162.075833 113.404136)
     (thickness 1.6)
-    (drawings 5)
-    (tracks 19)
+    (drawings 9)
+    (tracks 21)
     (zones 0)
     (modules 4)
@@
     (pad_drill 0.762)
     (pad_to_mask_clearance 0.2)
+    (solder_mask_min_width 0.25)
     (aux_axis_origin 144.78 108.585)
-    (visible_elements FFFFFF7F)
+    (visible_elements 7FFFFFFF)
     (pcbplotparams
-      (layerselection 0x010f0_80000001)
+      (layerselection 0x010f0_ffffffff)
       (usegerberextensions true)
+      (usegerberattributes false)
+      (usegerberadvancedattributes false)
+      (creategerberjobfile false)
       (excludeedgelayer true)
       (linewidth 0.100000)
@@
       (hpglpennumber 1)
       (hpglpenspeed 20)
-      (hpglpendiameter 15)
-      (hpglpenoverlay 2)
+      (hpglpendiameter 15.000000)
       (psnegative false)
       (psa4output false)
@@
       (drillshape 0)
       (scaleselection 1)
-      (outputdirectory gerber_single/))
+      (outputdirectory "gerbers/"))
   )
   (net 0 "")
@@
       (net 2 "Net-(F1-Pad1)"))
   )
+  (gr_arc (start 148.59 96.139) (end 148.59 95.504) (angle -180) (layer Edge.Cuts) (width 0.15))
+  (gr_arc (start 159.893 96.139) (end 159.893 96.774) (angle -180) (layer Edge.Cuts) (width 0.15))
+  (gr_line (start 159.893 96.774) (end 148.59 96.774) (layer Edge.Cuts) (width 0.15))
+  (gr_line (start 148.59 95.504) (end 159.893 95.504) (layer Edge.Cuts) (width 0.15))
   (gr_line (start 144.78 108.585) (end 145.415 108.585) (angle 90) (layer Edge.Cuts) (width 0.15))
   (gr_line (start 144.78 78.105) (end 144.78 108.585) (angle 90) (layer Edge.Cuts) (width 0.15))
@@
   (segment (start 156.8685 91.8845) (end 152.53 91.8845) (width 2) (layer B.Cu) (net 6) (status 400000))
   (segment (start 152.53 91.8845) (end 150.8155 93.599) (width 2) (layer B.Cu) (net 6) (status 800000))
+  (segment (start 156.8685 91.8845) (end 152.53 91.8845) (width 2) (layer F.Cu) (net 6) (status 400000))
+  (segment (start 152.53 91.8845) (end 150.8155 93.599) (width 2) (layer F.Cu) (net 6) (status 800000))
 )
