File: devices/Inline_SSR/Inline_SSR.sch (KiCad schematic (older format))
At the start: 4 parts, among them J1 JACK_STEREO, P1 CONN_01X02, U1 G3MB_SSR

Commit message: Big cleanup/upgrade of Kicad files
Parts:
- F1: symbol FUSE -> Inline_SSR-rescue:FUSE
- J1: symbol JACK_STEREO -> JACK_STEREO:JACK_STEREO
- P1: symbol CONN_01X02 -> conn:CONN_01X02
- U1: symbol G3MB_SSR -> G3MB-SSR:G3MB_SSR
Changed lines of the file:
@@
-EESchema Schematic File Version 2
-LIBS:power
-LIBS:device
-LIBS:transistors
-LIBS:conn
-LIBS:linear
-LIBS:regul
-LIBS:74xx
-LIBS:cmos4000
-LIBS:adc-dac
-LIBS:memory
-LIBS:xilinx
-LIBS:microcontrollers
-LIBS:dsp
-LIBS:microchip
-LIBS:analog_switches
-LIBS:motorola
-LIBS:texas
-LIBS:intel
-LIBS:audio
-LIBS:interface
-LIBS:digital-audio
-LIBS:philips
-LIBS:display
-LIBS:cypress
-LIBS:siliconi
-LIBS:opto
-LIBS:atmel
-LIBS:contrib
-LIBS:valves
-LIBS:G3MB-SSR
-LIBS:JACK_STEREO
-EELAYER 25 0
+EESchema Schematic File Version 4
+LIBS:Inline_SSR-cache
+EELAYER 26 0
 EELAYER END
 $Descr A4 11693 8268
@@
 $EndDescr
 $Comp
-L JACK_STEREO J1
+L JACK_STEREO:JACK_STEREO J1
 U 1 1 5932639C
 P 3600 3250
@@
 $EndComp
 $Comp
-L G3MB_SSR U1
+L G3MB-SSR:G3MB_SSR U1
 U 1 1 593263CF
 P 5100 3200
@@
 	4300 3000 4450 3000
 $Comp
-L FUSE F1
+L Inline_SSR-rescue:FUSE F1
 U 1 1 5932647D
 P 6050 3000
@@
 	5700 3000 5800 3000
 $Comp
-L CONN_01X02 P1
+L conn:CONN_01X02 P1
 U 1 1 593264D9
 P 6600 3050
