File: devices/SoManySwitches-ClientBoard/SoManySwitches-ClientBoard.sch (KiCad schematic (older format))
At the start: 8 parts, among them J1 RJ45, P1 CONN_02X06

Commit message: Big cleanup/upgrade of Kicad files
Parts:
- J1: symbol RJ45 -> conn:RJ45
- P1: symbol CONN_02X06 -> conn:CONN_02X06
- R1, R2: symbol R -> Device:R
- RP1, RP2, RP3, RP4: symbol R_PACK4 -> SoManySwitches-ClientBoard-rescue:R_PACK4
Changed lines of the file:
@@
-EESchema Schematic File Version 2
-LIBS:power
-LIBS:device
-LIBS:transistors
-LIBS:conn
-LIBS:linear
-LIBS:regul
-LIBS:74xx
-LIBS:cmos4000
-LIBS:adc-dac
-LIBS:memory
-LIBS:xilinx
-LIBS:microcontrollers
-LIBS:dsp
-LIBS:microchip
-LIBS:analog_switches
-LIBS:motorola
-LIBS:texas
-LIBS:intel
-LIBS:audio
-LIBS:interface
-LIBS:digital-audio
-LIBS:philips
-LIBS:display
-LIBS:cypress
-LIBS:siliconi
-LIBS:opto
-LIBS:atmel
-LIBS:contrib
-LIBS:valves
-EELAYER 25 0
+EESchema Schematic File Version 4
+LIBS:SoManySwitches-ClientBoard-cache
+EELAYER 26 0
 EELAYER END
 $Descr A4 11693 8268
@@
 $EndDescr
 $Comp
-L RJ45 J1
+L conn:RJ45 J1
 U 1 1 59240783
 P 3900 2350
@@
 $EndComp
 $Comp
-L GND #PWR01
+L power:GND #PWR01
 U 1 1 592407BA
 P 3550 2900
@@
 $EndComp
 $Comp
-L +5V #PWR02
+L power:+5V #PWR02
 U 1 1 592407D0
 P 4450 2750
@@
 	3550 2800 3550 2900
 $Comp
-L R R1
+L Device:R R1
 U 1 1 59240807
 P 5450 1950
@@
 $EndComp
 $Comp
-L R R2
+L Device:R R2
 U 1 1 5924083C
 P 5450 2450
@@
 $EndComp
 Wire Wire Line
-	5450 2300 5450 2100
+	5450 2300 5450 2200
 Wire Wire Line
 	5450 2200 5700 2200
@@
 Connection ~ 5450 2200
 $Comp
-L +3.3V #PWR03
+L power:+3.3V #PWR03
 U 1 1 5924088F
 P 5700 2150
@@
 $EndComp
 $Comp
-L +5V #PWR04
+L power:+5V #PWR04
 U 1 1 592408AA
 P 5450 1750
@@
 $EndComp
 $Comp
-L GND #PWR05
+L power:GND #PWR05
 U 1 1 592408BE
 P 5450 2700
@@
 	5450 1800 5450 1750
 $Comp
-L R_PACK4 RP1
+L SoManySwitches-ClientBoard-rescue:R_PACK4 RP1
 U 1 1 5924091D
 P 3600 3300
@@
 $EndComp
 $Comp
-L R_PACK4 RP3
+L SoManySwitches-ClientBoard-rescue:R_PACK4 RP3
 U 1 1 5924096A
 P 4200 3300
@@
 	4250 2950 4250 3100
 $Comp
-L R_PACK4 RP2
+L SoManySwitches-ClientBoard-rescue:R_PACK4 RP2
 U 1 1 59240A3C
 P 3600 4150
@@
 $EndComp
 $Comp
-L R_PACK4 RP4
+L SoManySwitches-ClientBoard-rescue:R_PACK4 RP4
 U 1 1 59240A6A
 P 4200 4150
@@
 $EndComp
 Wire Wire Line
-	4350 3950 4350 3500
-Wire Wire Line
-	4250 3950 4250 3500
-Wire Wire Line
-	3950 3950 3950 3500
-Wire Wire Line
-	3850 3950 3850 3500
-Wire Wire Line
-	3750 3950 3750 3500
-Wire Wire Line
-	3650 3950 3650 3500
+	4350 3950 4350 3900
+Wire Wire Line
+	4250 3950 4250 3850
+Wire Wire Line
+	3950 3950 3950 3800
+Wire Wire Line
+	3850 3950 3850 3750
+Wire Wire Line
+	3750 3950 3750 3700
+Wire Wire Line
+	3650 3950 3650 3650
 Wire Wire Line
 	4350 3900 4750 3900
@@
 Connection ~ 3650 3650
 $Comp
-L GND #PWR06
+L power:GND #PWR06
 U 1 1 59240CEE
 P 3650 4500
@@
 $EndComp
 Wire Wire Line
-	3650 4350 3650 4500
-Wire Wire Line
-	3650 4450 4550 4450
+	3650 4350 3650 4450
+Wire Wire Line
+	3650 4450 3750 4450
 Wire Wire Line
 	4550 4450 4550 4350
@@
 Connection ~ 3750 4450
 $Comp
-L CONN_02X06 P1
+L conn:CONN_02X06 P1
 U 1 1 59240EBF
 P 5300 3700
@@
 	5550 3450 5600 3450
 Wire Wire Line
-	5600 3300 5600 3950
-$Comp
-L +3.3V #PWR07
+	5600 3300 5600 3450
+$Comp
+L power:+3.3V #PWR07
 U 1 1 5924119A
 P 5600 3300
@@
 	5550 3850 5600 3850
 Connection ~ 5600 3850
+Wire Wire Line
+	5450 2200 5450 2100
+Wire Wire Line
+	4350 3900 4350 3500
+Wire Wire Line
+	4250 3850 4250 3500
+Wire Wire Line
+	3950 3800 3950 3500
+Wire Wire Line
+	3850 3750 3850 3500
+Wire Wire Line
+	3750 3700 3750 3500
+Wire Wire Line
+	3650 3650 3650 3500
+Wire Wire Line
+	3650 4450 3650 4500
+Wire Wire Line
+	4450 4450 4550 4450
+Wire Wire Line
+	4350 4450 4450 4450
+Wire Wire Line
+	4250 4450 4350 4450
+Wire Wire Line
+	3950 4450 4250 4450
+Wire Wire Line
+	3850 4450 3950 4450
+Wire Wire Line
+	3750 4450 3850 4450
+Wire Wire Line
+	5600 3450 5600 3550
+Wire Wire Line
+	5600 3550 5600 3650
+Wire Wire Line
+	5600 3650 5600 3750
+Wire Wire Line
+	5600 3750 5600 3850
+Wire Wire Line
+	5600 3850 5600 3950
 $EndSCHEMATC
