File: devices/4Channel_RGBW_LED_Controller/1Wire-LEDController.kicad_pcb (KiCad board)
At the start: 2 copper layers, 99.8 x 99.8 mm, 40 parts, among them CON1 BARREL_JACK, J1 RJ45, J2 RJ45, J3 JACK_STEREO, P1 CONN_02X05, P2 CONN_01X05, P3 CONN_01X05, P4 DC_IN, P5 CONN_01X05, P6 CONN_01X05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

Commit message: Bump all active boards to Revision 1.2
- Remove dropping resistor from 5V power line
- Add pullup resistor to Reset line
- Add pin markings to STM32 chip footprint

Signed-off-by: Alastair D'Silva <alastair@d-silva.org>
Parts:
- removed G***: OSHW-logo_silkscreen-front_4mm, OSHW Logo:OSHW-logo_silkscreen-front_4mm
- removed REF1, REF2, REF3, REF4: MountingHole_3.2mm_M3, Mounting_Holes:MountingHole_3.2mm_M3
- R1: value 33R -> 10k
- moved R1 17.7 mm to (171.9, 126.5), turned to 180 degrees
Connections:
- C1 pad 1: Net-(C1-Pad1) -> +5V
- P1 pad 6: (no net) -> Net-(P1-Pad6)
- P1 pad 7: (no net) -> Net-(P1-Pad7)
- P1 pad 8: (no net) -> Net-(P1-Pad8)
- Q1 pad 1: /CHAN2_R -> /CHAN2_W
- Q10 pad 1: /CHAN0_R -> /CHAN0_W
- Q11 pad 1: /CHAN3_G -> /CHAN3_B
- Q12 pad 1: /CHAN0_G -> /CHAN0_B
- Q13 pad 1: /CHAN3_B -> /CHAN3_R
- Q14 pad 1: /CHAN0_B -> /CHAN0_R
- Q15 pad 1: /CHAN3_W -> /CHAN3_G
- Q16 pad 1: /CHAN0_W -> /CHAN0_G
- Q2 pad 1: /CHAN2_G -> /CHAN2_B
- Q3 pad 1: /CHAN1_R -> /CHAN1_W
- Q4 pad 1: /CHAN2_B -> /CHAN2_R
- Q5 pad 1: /CHAN1_G -> /CHAN1_B
- Q6 pad 1: /CHAN2_W -> /CHAN2_G
- Q7 pad 1: /CHAN1_B -> /CHAN1_R
- Q8 pad 1: /CHAN1_W -> /CHAN1_G
- Q9 pad 1: /CHAN3_R -> /CHAN3_W
- R1 pad 1: +5V -> +3V3
- R1 pad 2: Net-(C1-Pad1) -> Net-(P1-Pad10)
- U1 pad 1: Net-(C1-Pad1) -> +5V
- U2 pad 11: (no net) -> Net-(U2-Pad11)
- U2 pad 14: (no net) -> Net-(U2-Pad14)
- U2 pad 15: (no net) -> Net-(U2-Pad15)
- U2 pad 18: (no net) -> Net-(U2-Pad18)
- U2 pad 19: (no net) -> Net-(U2-Pad19)
- U2 pad 2: (no net) -> Net-(U2-Pad2)
- U2 pad 20: (no net) -> Net-(U2-Pad20)
- U2 pad 21: (no net) -> Net-(U2-Pad21)
- U2 pad 22: (no net) -> Net-(U2-Pad22)
- U2 pad 23: /CHAN3_W -> /CHAN3_G
- U2 pad 24: (no net) -> Net-(U2-Pad24)
- U2 pad 25: /CHAN3_B -> /CHAN3_R
- U2 pad 26: (no net) -> Net-(U2-Pad26)
- U2 pad 27: /CHAN3_G -> /CHAN3_B
- U2 pad 28: (no net) -> Net-(U2-Pad28)
- U2 pad 29: /CHAN3_R -> /CHAN3_W
- U2 pad 3: (no net) -> Net-(U2-Pad3)
- U2 pad 30: (no net) -> Net-(U2-Pad30)
- U2 pad 33: /CHAN2_W -> /CHAN2_G
- U2 pad 34: /CHAN2_B -> /CHAN2_R
- U2 pad 35: (no net) -> Net-(U2-Pad35)
- U2 pad 36: /CHAN2_G -> /CHAN2_B
- U2 pad 37: (no net) -> Net-(U2-Pad37)
- U2 pad 38: /CHAN2_R -> /CHAN2_W
- U2 pad 39: (no net) -> Net-(U2-Pad39)
- U2 pad 4: (no net) -> Net-(U2-Pad4)
- U2 pad 40: /CHAN1_W -> /CHAN1_G
- U2 pad 41: (no net) -> Net-(U2-Pad41)
- U2 pad 42: /CHAN1_B -> /CHAN1_R
- U2 pad 43: (no net) -> Net-(U2-Pad43)
- U2 pad 44: /CHAN1_G -> /CHAN1_B
- U2 pad 45: (no net) -> Net-(U2-Pad45)
- U2 pad 47: (no net) -> Net-(U2-Pad47)
- U2 pad 48: /CHAN1_R -> /CHAN1_W
- U2 pad 50: (no net) -> Net-(U2-Pad50)
- U2 pad 51: (no net) -> Net-(U2-Pad51)
- U2 pad 52: (no net) -> Net-(U2-Pad52)
- U2 pad 53: /CHAN0_W -> /CHAN0_G
- U2 pad 55: /CHAN0_B -> /CHAN0_R
- U2 pad 56: (no net) -> Net-(U2-Pad56)
- U2 pad 57: /CHAN0_G -> /CHAN0_B
- U2 pad 58: (no net) -> Net-(U2-Pad58)
- U2 pad 59: /CHAN0_R -> /CHAN0_W
- U2 pad 6: (no net) -> Net-(U2-Pad6)
- U2 pad 61: (no net) -> Net-(U2-Pad61)
- U2 pad 62: (no net) -> Net-(U2-Pad62)
- U2 pad 8: (no net) -> Net-(U2-Pad8)
- U2 pad 9: (no net) -> Net-(U2-Pad9)
Routing:
- net /CHAN2_W: track 31.0 -> 13.4 mm, vias 1 -> 0
- net Net-(C1-Pad1): track 14.5 -> 0.00 mm
- net +5V: track 68.2 -> 81.2 mm
- net +3V3: track 139.5 -> 151.7 mm
- net /CHAN1_W: track 11.4 -> 23.5 mm, vias 1 -> 0
- net /CHAN2_G: track 21.0 -> 31.0 mm
- net /CHAN2_R: track 13.4 -> 23.0 mm
- net /CHAN1_R: track 23.5 -> 14.9 mm
- net /CHAN0_R: track 23.3 -> 19.2 mm
- net /CHAN3_W: track 23.0 -> 19.4 mm, vias 1 -> 0
- net Net-(P1-Pad10): track 25.0 -> 28.4 mm
- net /CHAN0_G: track 19.7 -> 22.2 mm
- net /CHAN1_G: track 13.8 -> 11.4 mm
- net /CHAN3_G: track 20.8 -> 23.0 mm
- net /CHAN3_B: track 18.7 -> 20.8 mm, vias 0 -> 1
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Other:
- board text added: "1Wire LED Controller Rev 1.2"
- board text added: "Licensed under the TAPR Open Hardware License (www.tapr.org/OHL) Copyright © 2018 Inferno Embedded"
- board text removed: "1Wire LED Controller Rev 2.1"
- board text removed: "Licensed under the TAPR Open Hardware License (www.tapr.org/OHL) Copyright © 2017 Inferno Embedded"
