File: devices/Aircon_Zone_Controller/1Wire-AC_Zoning.kicad_pcb (KiCad board)
At the start: 2 copper layers, 99.9 x 94.5 mm, 43 parts, among them CON1 BARREL_JACK, J1 RJ45, J2 RJ45, J3 JACK_STEREO, P1 CONN_02X05, P2 CONN_01X02, P6 CONN_01X05, U1 LP2950, U10 G3MB_SSR, U11 G3MB_SSR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

Commit message: Bump all active boards to Revision 1.2
- Remove dropping resistor from 5V power line
- Add pullup resistor to Reset line
- Add pin markings to STM32 chip footprint

Signed-off-by: Alastair D'Silva <alastair@d-silva.org>
Parts:
- removed H1, H2, H3, H4: MountingHole_3.2mm_M3, Mounting_Holes:MountingHole_3.2mm_M3
- moved R1 49.2 mm to (183.7, 107.7), turned to 180 degrees
Connections:
- C1 pad 1: Net-(C1-Pad1) -> +5V
- CON1 pad 2: (no net) -> Net-(CON1-Pad2)
- P1 pad 6: (no net) -> Net-(P1-Pad6)
- P1 pad 7: (no net) -> Net-(P1-Pad7)
- P1 pad 8: (no net) -> Net-(P1-Pad8)
- R1 pad 1: +5V -> +3V3
- R1 pad 2: Net-(C1-Pad1) -> Net-(P1-Pad10)
- U1 pad 1: Net-(C1-Pad1) -> +5V
- U2 pad 10: (no net) -> Net-(U2-Pad10)
- U2 pad 11: (no net) -> Net-(U2-Pad11)
- U2 pad 14: (no net) -> Net-(U2-Pad14)
- U2 pad 15: (no net) -> Net-(U2-Pad15)
- U2 pad 2: (no net) -> Net-(U2-Pad2)
- U2 pad 20: (no net) -> Net-(U2-Pad20)
- U2 pad 21: (no net) -> Net-(U2-Pad21)
- U2 pad 22: (no net) -> Net-(U2-Pad22)
- U2 pad 23: (no net) -> Net-(U2-Pad23)
- U2 pad 24: (no net) -> Net-(U2-Pad24)
- U2 pad 25: (no net) -> Net-(U2-Pad25)
- U2 pad 26: (no net) -> Net-(U2-Pad26)
- U2 pad 27: (no net) -> Net-(U2-Pad27)
- U2 pad 28: (no net) -> Net-(U2-Pad28)
- U2 pad 29: (no net) -> Net-(U2-Pad29)
- U2 pad 3: (no net) -> Net-(U2-Pad3)
- U2 pad 30: (no net) -> Net-(U2-Pad30)
- U2 pad 39: (no net) -> Net-(U2-Pad39)
- U2 pad 4: (no net) -> Net-(U2-Pad4)
- U2 pad 41: (no net) -> Net-(U2-Pad41)
- U2 pad 43: (no net) -> Net-(U2-Pad43)
- U2 pad 45: (no net) -> Net-(U2-Pad45)
- U2 pad 47: (no net) -> Net-(U2-Pad47)
- U2 pad 50: (no net) -> Net-(U2-Pad50)
- U2 pad 52: (no net) -> Net-(U2-Pad52)
- U2 pad 55: (no net) -> Net-(U2-Pad55)
- U2 pad 57: (no net) -> Net-(U2-Pad57)
- U2 pad 59: (no net) -> Net-(U2-Pad59)
- U2 pad 6: (no net) -> Net-(U2-Pad6)
- U2 pad 61: (no net) -> Net-(U2-Pad61)
- U2 pad 62: (no net) -> Net-(U2-Pad62)
- U2 pad 8: (no net) -> Net-(U2-Pad8)
- U2 pad 9: (no net) -> Net-(U2-Pad9)
- ZONE0 pad 1: (no net) -> Net-(ZONE0-Pad1)
- ZONE0 pad 8: (no net) -> Net-(ZONE0-Pad8)
- ZONE1 pad 1: (no net) -> Net-(ZONE1-Pad1)
- ZONE1 pad 8: (no net) -> Net-(ZONE1-Pad8)
- ZONE2 pad 1: (no net) -> Net-(ZONE2-Pad1)
- ZONE2 pad 8: (no net) -> Net-(ZONE2-Pad8)
- ZONE3 pad 1: (no net) -> Net-(ZONE3-Pad1)
- ZONE3 pad 8: (no net) -> Net-(ZONE3-Pad8)
- ZONE4 pad 1: (no net) -> Net-(ZONE4-Pad1)
- ZONE4 pad 8: (no net) -> Net-(ZONE4-Pad8)
- ZONE5 pad 1: (no net) -> Net-(ZONE5-Pad1)
- ZONE5 pad 8: (no net) -> Net-(ZONE5-Pad8)
- ZONE6 pad 1: (no net) -> Net-(ZONE6-Pad1)
- ZONE6 pad 8: (no net) -> Net-(ZONE6-Pad8)
- ZONE7 pad 1: (no net) -> Net-(ZONE7-Pad1)
- ZONE7 pad 8: (no net) -> Net-(ZONE7-Pad8)
Routing:
- net +5V: track 221.2 -> 236.1 mm
- net Net-(C1-Pad1): track 14.2 -> 0.00 mm
- net +3V3: track 82.3 -> 95.3 mm
- net Net-(P1-Pad10): track 34.0 -> 36.4 mm
Other:
- board text added: "1Wire 8 Zone AC Controller Rev 1.2"
- board text added: "Licensed under the TAPR Open Hardware License (www.tapr.org/OHL) Copyright © 2018 Inferno Embedded"
- board text removed: "1Wire 8 Zone AC Controller Rev 1.0"
- board text removed: "Licensed under the TAPR Open Hardware License (www.tapr.org/OHL) Copyright © 2017 Inferno Embedded"
