File: devices/SoManySwitches/1Wire-SoManySwitches.sch (KiCad schematic (older format))
At the start: 20 parts, among them J1 RJ45, J10 RJ45, J2 RJ45, J3 RJ45, J4 RJ45, J5 RJ45, J6 RJ45, J7 RJ45, J8 RJ45, J9 RJ45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

Commit message: Bump all active boards to Revision 1.2
- Remove dropping resistor from 5V power line
- Add pullup resistor to Reset line
- Add pin markings to STM32 chip footprint

Signed-off-by: Alastair D'Silva <alastair@d-silva.org>
Parts:
- C1: symbol CP -> 1Wire-SoManySwitches-rescue:CP
- C2, C3, C4, C5: symbol C -> 1Wire-SoManySwitches-rescue:C
- J1, J10, J2, J3, J4, J5, J6, J7, J8, J9: symbol RJ45 -> 1Wire-SoManySwitches-rescue:RJ45
- P1: symbol CONN_02X05 -> 1Wire-SoManySwitches-rescue:CONN_02X05
- P6: symbol CONN_01X05 -> 1Wire-SoManySwitches-rescue:CONN_01X05
- R1: value 33R -> 10K; symbol R -> 1Wire-SoManySwitches-rescue:R
- U1: symbol LP2950 -> 1Wire-SoManySwitches-rescue:LP2950
- U2: symbol STM32F030R8 -> 1Wire-SoManySwitches-rescue:STM32F030R8
Connections:
- net +3V3: now also R1.1
- net +5V: now also C1.1, U1.1 (VI); no longer J7.8, J8.8, R1.1
- net at P1.10 (P10), U2.7 (NRST): now also R1.2
- new net: J7.8, J8.8
Other:
- moved on the sheet: R1
